File: Schematic/Schematic/FreePublicBicycles.sch (KiCad schematic (older format))
At the start: 40 parts

Commit message: Added PCB design
Parts:
- removed BZ?: Buzzer, symbol Device:Buzzer
- removed C? (x2): 10n, symbol Device:C_Small
- removed D?: 1N4007, symbol Device:D_ALT
- removed Q?: 2N2222, symbol Device:Q_NPN_EBC
- removed R?: 25k, symbol Device:R
- added C?: 100n, symbol Device:C_Small
- added R?: 1k, symbol Device:R
- C?: footprint (none) -> Capacitor_THT:CP_Radial_D5.0mm_P2.00mm
- C?: value 100u -> 0.33u
- D?: footprint Diode_THT:D_DO-201AE_P15.24mm_Horizontal -> Diode_THT:D_DO-15_P15.24mm_Horizontal
Connections:
- net +3V3: now also C?.1; no longer C?.1
- net +5V: now also C?.1; no longer C?.1
- net BUTTON: now also R?.1; no longer SW?.1
- net GND: now also C?.2
- net RX: now also U?.14 (PB0); no longer U?.2 (PD0)
- net TX: now also U?.15 (PB1); no longer U?.3 (PD1)
- net BUZZER: no longer names the net of U?.24 (PC1)
- new net: C?.1, R?.2, SW?.1
- no-connect marks 4 -> 14
Other:
- moved on the sheet: C?, SW?
