File: Gateway_PCB/Gateway_Schematic.sch (KiCad schematic (older format))
At the start: 5 parts, among them J1 Conn_01x40_Female, J2 Conn_01x08_Female, J3 Conn_01x08_Female, J4 Conn_01x01_Female

Commit message: Changed RFM95W footprint and added SMA Connector Model
Parts:
- removed J2, J3: Conn_01x08_Female, Connector_PinSocket_2.00mm:PinSocket_1x08_P2.00mm_Vertical, symbol Connector:Conn_01x08_Female
- added U1: RFM95W-868S2, RFM95:XCVR_RFM95W-915S2, symbol RF_AM_FM:RFM95W-868S2
Connections:
- net +3V3: now also U1.13 (3.3V)
- net ANT: now also U1.9 (ANT)
- net DIO0: now also U1.14 (DIO0)
- net DIO1: now also U1.15 (DIO1)
- net GND: now also J1.20 (Pin_20), J1.39 (Pin_39), U1.1 (GND), U1.10 (GND), U1.8 (GND); no longer J1.9 (Pin_9)
- net MISO: now also U1.2 (MISO)
- net MOSI: now also U1.3 (MOSI)
- net NSS: now also U1.5 (NSS)
- net RST: now also U1.6 (RESET)
- net SCK: now also U1.4 (SCK)
- no-connect marks 7 -> 34
Other:
- moved on the sheet: J4
Changed lines of the file:
@@
 	1    0    0    -1
-$EndComp
-Wire Wire Line
-	2250 5500 2400 5500
-$Comp
-L power:GND #PWR01
-U 1 1 5E37C329
-P 2400 5500
-F 0 "#PWR01" H 2400 5250 50  0001 C CNN
-F 1 "GND" H 2550 5500 50  0000 C CNN
-F 2 "" H 2400 5500 50  0001 C CNN
-F 3 "" H 2400 5500 50  0001 C CNN
-	1    2400 5500
-	1    0    0    -1
-$EndComp
-$Comp
-L Connector:Conn_01x08_Female J2
-U 1 1 5E37EAFD
-P 6450 3900
-F 0 "J2" H 6477 3876 50  0000 L CNN
-F 1 "Conn_01x08_Female" H 6477 3785 50  0000 L CNN
-F 2 "Connector_PinSocket_2.00mm:PinSocket_1x08_P2.00mm_Vertical" H 6450 3900 50  0001 C CNN
-F 3 "~" H 6450 3900 50  0001 C CNN
-	1    6450 3900
-	1    0    0    -1
-$EndComp
-$Comp
-L power:+3.3V #PWR03
-U 1 1 5E3803B6
-P 6100 4000
-F 0 "#PWR03" H 6100 3850 50  0001 C CNN
-F 1 "+3.3V" H 5850 4050 50  0000 C CNN
-F 2 "" H 6100 4000 50  0001 C CNN
-F 3 "" H 6100 4000 50  0001 C CNN
-	1    6100 4000
-	1    0    0    -1
-$EndComp
-Wire Wire Line
-	6100 4000 6250 4000
-Wire Wire Line
-	7600 3600 7800 3600
-$Comp
-L power:GND #PWR04
-U 1 1 5E381581
-P 7800 3600
-F 0 "#PWR04" H 7800 3350 50  0001 C CNN
-F 1 "GND" H 7950 3550 50  0000 C CNN
-F 2 "" H 7800 3600 50  0001 C CNN
-F 3 "" H 7800 3600 50  0001 C CNN
-	1    7800 3600
-	1    0    0    -1
-$EndComp
-Wire Wire Line
-	7600 3800 7850 3800
-Text GLabel 7850 3800 2    50   Input ~ 0
-RST
-Wire Wire Line
-	7600 3900 7850 3900
-Text GLabel 7850 3900 2    50   Input ~ 0
-NSS
-Text GLabel 7850 4000 2    50   Input ~ 0
-SCK
-Wire Wire Line
-	7600 4100 7850 4100
-Text GLabel 7850 4100 2    50   Input ~ 0
-MOSI
-Wire Wire Line
-	7600 4000 7850 4000
-Wire Wire Line
-	7600 4200 7850 4200
-Text GLabel 7850 4200 2    50   Input ~ 0
-MISO
-NoConn ~ 6250 3800
-NoConn ~ 6250 3900
-NoConn ~ 6250 4100
-NoConn ~ 6250 4200
-NoConn ~ 6250 4300
-NoConn ~ 7600 3700
-Wire Wire Line
-	6250 3700 6050 3700
-$Comp
-L power:GND #PWR05
-U 1 1 5E38FD01
-P 6050 3700
-F 0 "#PWR05" H 6050 3450 50  0001 C CNN
-F 1 "GND" H 6200 3650 50  0000 C CNN
-F 2 "" H 6050 3700 50  0001 C CNN
-F 3 "" H 6050 3700 50  0001 C CNN
-	1    6050 3700
-	-1   0    0    -1
 $EndComp
 $Comp
 L Connector:Conn_01x01_Female J4
 U 1 1 5E390D2A
-P 5550 2950
-F 0 "J4" V 5490 2862 50  0000 R CNN
-F 1 "Conn_01x01_Female" V 5399 2862 50  0000 R CNN
-F 2 "Connector_Coaxial:SMA_Amphenol_901-144_Vertical" H 5550 2950 50  0001 C CNN
-F 3 "~" H 5550 2950 50  0001 C CNN
-	1    5550 2950
+P 8150 2050
+F 0 "J4" V 8090 1962 50  0000 R CNN
+F 1 "Conn_01x01_Female" V 7999 1962 50  0000 R CNN
+F 2 "Connector_Coaxial:SMA_Amphenol_901-144_Vertical" H 8150 2050 50  0001 C CNN
+F 3 "~" H 8150 2050 50  0001 C CNN
+	1    8150 2050
 	0    -1   -1   0
 $EndComp
 Wire Wire Line
-	6000 3600 6250 3600
-Text GLabel 6000 3600 0    50   Input ~ 0
-ANT
-Wire Wire Line
-	5550 3150 5550 3250
-Text GLabel 5550 3250 3    50   Input ~ 0
+	8150 2250 8150 2350
+Text GLabel 8150 2350 3    50   Input ~ 0
 ANT
 $Comp
-L Connector:Conn_01x08_Female J3
-U 1 1 5E37EB67
-P 7400 4000
-F 0 "J3" H 7294 3375 50  0000 C CNN
-F 1 "Conn_01x08_Female" H 7294 3466 50  0000 C CNN
-F 2 "Connector_PinSocket_2.00mm:PinSocket_1x08_P2.00mm_Vertical" H 7400 4000 50  0001 C CNN
-F 3 "~" H 7400 4000 50  0001 C CNN
-	1    7400 4000
+L RF_AM_FM:RFM95W-868S2 U1
+U 1 1 5E3934E9
+P 7000 3200
+F 0 "U1" H 6300 3800 50  0000 C CNN
+F 1 "RFM95W-868S2" H 6300 3700 50  0000 C CNN
+F 2 "RFM95:XCVR_RFM95W-915S2" H 3700 4850 50  0001 C CNN
+F 3 "http://www.hoperf.com/upload/rf/RFM95_96_97_98W.pdf" H 3700 4850 50  0001 C CNN
+	1    7000 3200
+	1    0    0    -1
+$EndComp
+$Comp
+L power:+3.3V #PWR0101
+U 1 1 5E393577
+P 7000 2650
+F 0 "#PWR0101" H 7000 2500 50  0001 C CNN
+F 1 "+3.3V" H 6750 2700 50  0000 C CNN
+F 2 "" H 7000 2650 50  0001 C CNN
+F 3 "" H 7000 2650 50  0001 C CNN
+	1    7000 2650
+	1    0    0    -1
+$EndComp
+Wire Wire Line
+	7000 2650 7000 2700
+Wire Wire Line
+	7750 2900 7500 2900
+Text GLabel 7750 2900 2    50   Input ~ 0
+ANT
+Text GLabel 6250 2900 0    50   Input ~ 0
+SCK
+Wire Wire Line
+	6500 2900 6250 2900
+Wire Wire Line
+	6500 3000 6250 3000
+Text GLabel 6250 3000 0    50   Input ~ 0
+MOSI
+Wire Wire Line
+	6500 3100 6250 3100
+Text GLabel 6250 3100 0    50   Input ~ 0
+MISO
+Wire Wire Line
+	6500 3200 6250 3200
+Text GLabel 6250 3200 0    50   Input ~ 0
+NSS
+$Comp
+L power:GND #PWR0102
+U 1 1 5E398A51
+P 6300 3600
+F 0 "#PWR0102" H 6300 3350 50  0001 C CNN
+F 1 "GND" H 6450 3550 50  0000 C CNN
+F 2 "" H 6300 3600 50  0001 C CNN
+F 3 "" H 6300 3600 50  0001 C CNN
+	1    6300 3600
 	-1   0    0    1
 $EndComp
-NoConn ~ 7600 4300
+Wire Wire Line
+	6500 3400 6250 3400
+Text GLabel 6250 3400 0    50   Input ~ 0
+RST
+Wire Wire Line
+	7500 3600 7750 3600
+Text GLabel 7750 3600 2    50   Input ~ 0
+DIO0
+Wire Wire Line
+	7500 3500 7750 3500
+Text GLabel 7750 3500 2    50   Input ~ 0
+DIO1
+NoConn ~ 7500 3400
+NoConn ~ 7500 3300
+NoConn ~ 7500 3200
+NoConn ~ 7500 3100
+Wire Wire Line
+	6900 3800 7000 3800
+Wire Wire Line
+	7000 3800 7100 3800
+Connection ~ 7000 3800
+Wire Wire Line
+	7000 3800 7000 3850
+$Comp
+L power:GND #PWR0103
+U 1 1 5E39C9C6
+P 7000 3850
+F 0 "#PWR0103" H 7000 3600 50  0001 C CNN
+F 1 "GND" H 7005 3677 50  0000 C CNN
+F 2 "" H 7000 3850 50  0001 C CNN
+F 3 "" H 7000 3850 50  0001 C CNN
+	1    7000 3850
+	1    0    0    -1
+$EndComp
+Wire Wire Line
+	2250 2500 2400 2500
+$Comp
+L power:GND #PWR0104
+U 1 1 5E39DA9D
+P 2400 2500
+F 0 "#PWR0104" H 2400 2250 50  0001 C CNN
+F 1 "GND" H 2550 2500 50  0000 C CNN
+F 2 "" H 2400 2500 50  0001 C CNN
+F 3 "" H 2400 2500 50  0001 C CNN
+	1    2400 2500
+	1    0    0    -1
+$EndComp
+NoConn ~ 2250 2400
+NoConn ~ 2250 2600
+NoConn ~ 2250 2700
+NoConn ~ 2250 2800
+NoConn ~ 2250 2900
+NoConn ~ 2250 3000
+NoConn ~ 2250 3100
+NoConn ~ 2250 3200
+NoConn ~ 2250 3300
+NoConn ~ 2250 3400
+NoConn ~ 2250 3500
+NoConn ~ 2250 3600
+NoConn ~ 2250 3700
+NoConn ~ 2250 3800
+NoConn ~ 2250 3900
+NoConn ~ 2250 4200
+NoConn ~ 2250 4600
+NoConn ~ 2250 4700
+NoConn ~ 2250 4800
+NoConn ~ 2250 5000
+NoConn ~ 2250 5100
+NoConn ~ 2250 5200
+NoConn ~ 2250 5400
+NoConn ~ 2250 5500
+NoConn ~ 2250 5600
+NoConn ~ 2250 5800
+NoConn ~ 2250 5900
+NoConn ~ 2250 6000
+NoConn ~ 2250 6100
+NoConn ~ 2250 6200
+Wire Wire Line
+	2250 4400 2400 4400
+$Comp
+L power:GND #PWR?
+U 1 1 5E3A3FD5
+P 2400 4400
+F 0 "#PWR?" H 2400 4150 50  0001 C CNN
+F 1 "GND" H 2550 4400 50  0000 C CNN
+F 2 "" H 2400 4400 50  0001 C CNN
+F 3 "" H 2400 4400 50  0001 C CNN
+	1    2400 4400
+	1    0    0    -1
+$EndComp
 $EndSCHEMATC
