File: Gateway_Schematic/Gateway_Schematic.sch (KiCad schematic (older format))
At the start: 4 parts, among them J1 Raspberry_Pi_2_3, U1 RFM95W-868S2

Commit message: Added changes to schematics
Other:
- note added: "Communication Unit"
- note added: "Control Unit"
- moved on the sheet: AE1, C1, U1
Changed lines of the file:
@@
 EESchema Schematic File Version 4
+LIBS:Gateway_Schematic-cache
 EELAYER 26 0
 EELAYER END
@@
 L RF_AM_FM:RFM95W-868S2 U1
 U 1 1 5E3753FD
-P 7700 3650
-F 0 "U1" H 7150 4350 50  0000 C CNN
-F 1 "RFM95W-868S2" H 7150 4250 50  0000 C CNN
-F 2 "" H 4400 5300 50  0001 C CNN
-F 3 "http://www.hoperf.com/upload/rf/RFM95_96_97_98W.pdf" H 4400 5300 50  0001 C CNN
-	1    7700 3650
-	1    0    0    -1
-$EndComp
-Wire Wire Line
-	7700 3150 7700 3100
-Wire Wire Line
-	7600 4250 7700 4250
-Connection ~ 7700 4250
-Wire Wire Line
-	7700 4250 7800 4250
-Wire Wire Line
-	7700 4250 7700 4300
+P 7700 3150
+F 0 "U1" H 7150 3850 50  0000 C CNN
+F 1 "RFM95W-868S2" H 7150 3750 50  0000 C CNN
+F 2 "" H 4400 4800 50  0001 C CNN
+F 3 "http://www.hoperf.com/upload/rf/RFM95_96_97_98W.pdf" H 4400 4800 50  0001 C CNN
+	1    7700 3150
+	1    0    0    -1
+$EndComp
+Wire Wire Line
+	7700 2650 7700 2600
+Wire Wire Line
+	7600 3750 7700 3750
+Connection ~ 7700 3750
+Wire Wire Line
+	7700 3750 7800 3750
+Wire Wire Line
+	7700 3750 7700 3800
 $Comp
 L power:+3.3V #PWR04
 U 1 1 5E375DB2
-P 7700 3100
-F 0 "#PWR04" H 7700 2950 50  0001 C CNN
-F 1 "+3.3V" H 7715 3273 50  0000 C CNN
-F 2 "" H 7700 3100 50  0001 C CNN
-F 3 "" H 7700 3100 50  0001 C CNN
-	1    7700 3100
+P 7700 2600
+F 0 "#PWR04" H 7700 2450 50  0001 C CNN
+F 1 "+3.3V" H 7715 2773 50  0000 C CNN
+F 2 "" H 7700 2600 50  0001 C CNN
+F 3 "" H 7700 2600 50  0001 C CNN
+	1    7700 2600
 	1    0    0    -1
 $EndComp
@@
 L power:GND #PWR05
 U 1 1 5E375E01
-P 7700 4300
-F 0 "#PWR05" H 7700 4050 50  0001 C CNN
-F 1 "GND" H 7705 4127 50  0000 C CNN
-F 2 "" H 7700 4300 50  0001 C CNN
-F 3 "" H 7700 4300 50  0001 C CNN
-	1    7700 4300
+P 7700 3800
+F 0 "#PWR05" H 7700 3550 50  0001 C CNN
+F 1 "GND" H 7705 3627 50  0000 C CNN
+F 2 "" H 7700 3800 50  0001 C CNN
+F 3 "" H 7700 3800 50  0001 C CNN
+	1    7700 3800
 	1    0    0    -1
 $EndComp
@@
 L Device:Antenna AE1
 U 1 1 5E375EFB
-P 8250 3100
-F 0 "AE1" H 8330 3091 50  0000 L CNN
-F 1 "Antenna" H 8330 3000 50  0000 L CNN
-F 2 "" H 8250 3100 50  0001 C CNN
-F 3 "~" H 8250 3100 50  0001 C CNN
-	1    8250 3100
-	1    0    0    -1
-$EndComp
-Wire Wire Line
-	8200 3350 8250 3350
-Wire Wire Line
-	8250 3350 8250 3300
+P 8250 2600
+F 0 "AE1" H 8330 2591 50  0000 L CNN
+F 1 "Antenna" H 8330 2500 50  0000 L CNN
+F 2 "" H 8250 2600 50  0001 C CNN
+F 3 "~" H 8250 2600 50  0001 C CNN
+	1    8250 2600
+	1    0    0    -1
+$EndComp
+Wire Wire Line
+	8200 2850 8250 2850
+Wire Wire Line
+	8250 2850 8250 2800
+Wire Wire Line
+	7200 2850 6950 2850
+Text GLabel 6950 2850 0    50   Input ~ 0
+SCK
+Wire Wire Line
+	7200 2950 6950 2950
+Text GLabel 6950 2950 0    50   Input ~ 0
+MOSI
+Wire Wire Line
+	7200 3050 6950 3050
+Text GLabel 6950 3050 0    50   Input ~ 0
+MISO
+Wire Wire Line
+	7200 3150 6950 3150
+Text GLabel 6950 3150 0    50   Input ~ 0
+NSS
 Wire Wire Line
 	7200 3350 6950 3350
 Text GLabel 6950 3350 0    50   Input ~ 0
-SCK
-Wire Wire Line
-	7200 3450 6950 3450
-Text GLabel 6950 3450 0    50   Input ~ 0
-MOSI
-Wire Wire Line
-	7200 3550 6950 3550
-Text GLabel 6950 3550 0    50   Input ~ 0
-MISO
-Wire Wire Line
-	7200 3650 6950 3650
-Text GLabel 6950 3650 0    50   Input ~ 0
-NSS
-Wire Wire Line
-	7200 3850 6950 3850
-Text GLabel 6950 3850 0    50   Input ~ 0
 RST
 Wire Wire Line
-	8200 4050 8450 4050
-Text GLabel 8450 4050 2    50   Input ~ 0
+	8200 3550 8450 3550
+Text GLabel 8450 3550 2    50   Input ~ 0
 DIO0
 Wire Wire Line
-	8200 3950 8450 3950
-Text GLabel 8450 3950 2    50   Input ~ 0
+	8200 3450 8450 3450
+Text GLabel 8450 3450 2    50   Input ~ 0
 DIO1
-NoConn ~ 8200 3850
-NoConn ~ 8200 3750
-NoConn ~ 8200 3650
-NoConn ~ 8200 3550
+NoConn ~ 8200 3350
+NoConn ~ 8200 3250
+NoConn ~ 8200 3150
+NoConn ~ 8200 3050
 $Comp
 L Device:C_Small C1
 U 1 1 5E37AEF1
-P 8850 2900
-F 0 "C1" H 8942 2946 50  0000 L CNN
-F 1 "100n" H 8942 2855 50  0000 L CNN
-F 2 "" H 8850 2900 50  0001 C CNN
-F 3 "~" H 8850 2900 50  0001 C CNN
-	1    8850 2900
-	1    0    0    -1
-$EndComp
-Wire Wire Line
-	8850 2800 8850 2750
-Wire Wire Line
-	8850 3000 8850 3050
+P 9000 2900
+F 0 "C1" H 9092 2946 50  0000 L CNN
+F 1 "100n" H 9092 2855 50  0000 L CNN
+F 2 "" H 9000 2900 50  0001 C CNN
+F 3 "~" H 9000 2900 50  0001 C CNN
+	1    9000 2900
+	1    0    0    -1
+$EndComp
+Wire Wire Line
+	9000 2800 9000 2750
+Wire Wire Line
+	9000 3000 9000 3050
 $Comp
 L power:+3.3V #PWR06
 U 1 1 5E37BB65
-P 8850 2750
-F 0 "#PWR06" H 8850 2600 50  0001 C CNN
-F 1 "+3.3V" H 8865 2923 50  0000 C CNN
-F 2 "" H 8850 2750 50  0001 C CNN
-F 3 "" H 8850 2750 50  0001 C CNN
-	1    8850 2750
+P 9000 2750
+F 0 "#PWR06" H 9000 2600 50  0001 C CNN
+F 1 "+3.3V" H 9015 2923 50  0000 C CNN
+F 2 "" H 9000 2750 50  0001 C CNN
+F 3 "" H 9000 2750 50  0001 C CNN
+	1    9000 2750
 	1    0    0    -1
 $EndComp
@@
 L power:GND #PWR07
 U 1 1 5E37BBA4
-P 8850 3050
-F 0 "#PWR07" H 8850 2800 50  0001 C CNN
-F 1 "GND" H 8855 2877 50  0000 C CNN
-F 2 "" H 8850 3050 50  0001 C CNN
-F 3 "" H 8850 3050 50  0001 C CNN
-	1    8850 3050
-	1    0    0    -1
-$EndComp
+P 9000 3050
+F 0 "#PWR07" H 9000 2800 50  0001 C CNN
+F 1 "GND" H 9005 2877 50  0000 C CNN
+F 2 "" H 9000 3050 50  0001 C CNN
+F 3 "" H 9000 3050 50  0001 C CNN
+	1    9000 3050
+	1    0    0    -1
+$EndComp
+Wire Notes Line
+	3100 2250 3100 5950
+Wire Notes Line
+	3100 5950 6000 5950
+Wire Notes Line
+	6000 5950 6000 2250
+Wire Notes Line
+	6000 2250 3100 2250
+Wire Notes Line
+	6300 4600 9450 4600
+Wire Notes Line
+	9450 4600 9450 2250
+Wire Notes Line
+	9450 2250 6300 2250
+Wire Notes Line
+	6300 2250 6300 4600
+Text Notes 3600 5800 0    200  ~ 0
+Control Unit
+Text Notes 6350 4400 0    200  ~ 0
+Communication Unit
 $EndSCHEMATC
