File: Transmitter_PCB/PCB.sch (KiCad schematic (older format))
At the start: 48 parts, among them J1 Conn_01x04_Female, J11 Conn_01x01_Female, J12 Conn_01x04_Female, J13 Conn_01x04_Female, J2 Conn_01x28_Female, J3 Conn_01x03_Female, J8 Conn_01x02_Female, J9 Conn_01x03_Female, Q1 PN2222A, Q2 IRF4905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

Commit message: Changed message identification
Parts:
- BT1: footprint Library:Battery_Holder -> (none)
- C1, C11, C14, C15, C16, C17, C19, C2, C5, C8: footprint Capacitor_THT:C_Disc_D3.0mm_W2.0mm_P2.50mm -> (none)
- C10, C12, C13, C18, C7: footprint Capacitor_THT:CP_Radial_D5.0mm_P2.00mm -> (none)
- C3, C4: footprint Capacitor_THT:C_Disc_D5.0mm_W2.5mm_P2.50mm -> (none)
- C6: footprint Capacitor_THT:CP_Radial_D10.0mm_P5.00mm -> (none)
- C9: footprint Capacitor_THT:C_Disc_D5.0mm_W2.5mm_P5.00mm -> (none)
- D1, D2, D3, D4: footprint Diode_THT:D_DO-41_SOD81_P10.16mm_Horizontal -> (none)
- D5: footprint Diode_THT:D_DO-15_P15.24mm_Horizontal -> Diode_THT:D_DO-201AE_P15.24mm_Horizontal
- H1, H2, H3, H4: footprint MountingHole:MountingHole_3.5mm_Pad_Via -> (none)
- J1: footprint Connector_Molex:Molex_KK-396_A-41791-0004_1x04_P3.96mm_Vertical -> (none)
- J11: footprint Connector_Coaxial:SMA_Amphenol_901-144_Vertical -> (none)
- J12, J13: footprint Connector_PinSocket_2.54mm:PinSocket_1x04_P2.54mm_Vertical -> (none)
- J2: footprint Package_DIP:DIP-28_W7.62mm -> (none)
- J8: footprint Connector_Molex:Molex_KK-254_AE-6410-02A_1x02_P2.54mm_Vertical -> (none)
- J9: footprint Connector_PinSocket_2.54mm:PinSocket_1x03_P2.54mm_Vertical -> (none)
- R1, R2, R3, R4, R5: footprint Resistor_THT:R_Axial_DIN0207_L6.3mm_D2.5mm_P10.16mm_Horizontal -> (none)
- U2: footprint MyComponents:MP1584 -> (none)
- Y1: footprint Crystal:Crystal_HC49-U_Vertical -> (none)
Other:
- moved on the sheet: H1, H2, H3, H4
